File: standalone_board/kicad/freqcounter_16F18446.sch (KiCad schematic (older format))
At the start: 41 parts, among them J1 ICSP, J2 UART, J3 INPUT CLK, J4 INPUT A, J5 INPUT B, J6 INPUT ZCD, J7 POWER, J8 ICSP2, P1 LCD_DISPLAY_16X2, U1 PIC16F18446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

Commit message: Bugfix schematic and PCB
Parts:
- removed C6: 100nF, Capacitor_SMD:C_0805_2012Metric_Pad1.15x1.40mm_HandSolder, symbol Device:C
- added R14: 2K2, Resistor_SMD:R_0805_2012Metric_Pad1.15x1.40mm_HandSolder, symbol Device:R
- U3: footprint (none) -> Package_SO:SOIC-14_3.9x8.7mm_P1.27mm
Connections:
- net Earth: now also R14.2
- net Vee: now also R14.1
Changed lines of the file:
@@
 Vee
-$Comp
-L Device:C C6
-U 1 1 5E722B3A
-P 3700 4150
-F 0 "C6" H 3815 4197 50  0000 L CNN
-F 1 "100nF" H 3815 4104 50  0000 L CNN
-F 2 "Capacitor_SMD:C_0805_2012Metric_Pad1.15x1.40mm_HandSolder" H 3738 4000 50  0001 C CNN
-F 3 "~" H 3700 4150 50  0001 C CNN
-	1    3700 4150
-	1    0    0    -1
-$EndComp
 $Comp
 L power:Earth #PWR05
@@
 F 0 "U3" H 2800 5523 50  0000 C CNN
 F 1 "PIC16F15325" H 2800 5430 50  0000 C CNN
-F 2 "" H 2800 5350 50  0001 C CNN
+F 2 "Package_SO:SOIC-14_3.9x8.7mm_P1.27mm" H 2800 5350 50  0001 C CNN
 F 3 "" H 2800 5350 50  0001 C CNN
 	1    2800 5350
@@
 Wire Wire Line
 	4400 2100 4400 2000
+$Comp
+L Device:R R14
+U 1 1 5EA9F859
+P 3700 4150
+F 0 "R14" H 3770 4197 50  0000 L CNN
+F 1 "2K2" H 3770 4104 50  0000 L CNN
+F 2 "Resistor_SMD:R_0805_2012Metric_Pad1.15x1.40mm_HandSolder" V 3630 4150 50  0001 C CNN
+F 3 "~" H 3700 4150 50  0001 C CNN
+	1    3700 4150
+	1    0    0    -1
+$EndComp
 $EndSCHEMATC
