File: arduino_shield/kicad/freqcounter.kicad_pcb (KiCad board)
At the start: 2 copper layers, 47 x 53.3 mm, 27 parts, among them J1 ICSP PICKIT, J10 INPUT_A, J11 INPUT_B, J12 INPUT_ZCD, J13 I2C_1, J14 I2C_2, J15 PARALEL, J2 Arduino_Power, J3 Arduino_Power, J4 Arduino_Digital_2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

Commit message: Arduino Shield PCB designed
Parts:
- added R5: 10K, Resistor_SMD:R_0805_2012Metric_Pad1.15x1.40mm_HandSolder, F.Cu at (144.8, 70.9)
- added R6: 10K, Resistor_SMD:R_0805_2012Metric_Pad1.15x1.40mm_HandSolder, F.Cu at (147.3, 70.9)
- J5, J8: footprint Footprints:Connector_1x06 -> Footprints:Connector_1x08
- J6: footprint Footprints:Connector_1x04 -> Footprints:Connector_1x06
- moved R2 85.9 mm to (135.6, 66.7), turned to 180 degrees
- moved R4 80.5 mm to (152.4, 78.1)
- moved R1 77.2 mm to (160.0, 78.7), turned to 180 degrees
- moved R3 73.3 mm to (146.9, 76.2)
- moved C3 63.6 mm to (152.4, 80.0)
- moved D1 50.1 mm to (147.3, 78.7), turned to 180 degrees
- moved J5 3.56 mm to (124.5, 62.2)
- moved J1 1.91 mm to (124.5, 90.2)
- moved J15 1.91 mm to (124.5, 85.1)
- moved J10 1.27 mm to (160.0, 97.8)
- moved J11 1.27 mm to (160.0, 90.2)
- moved J12 1.27 mm to (160.0, 82.5)
- moved J13 1.27 mm to (160.0, 67.3)
- moved J14 1.27 mm to (152.4, 67.3)
Connections:
- J1 pad 2: VDD -> 5V
- J13 pad 3: VDD -> 5V
- J14 pad 3: VDD -> 5V
- J15 pad 1: VDD -> 5V
- J5 pad 1: Net-(J4-Pad3) -> Net-(J4-Pad1)
- J5 pad 2: Net-(J4-Pad4) -> GND
- J5 pad 3: Net-(J4-Pad5) -> Net-(J4-Pad3)
- J5 pad 4: Net-(J4-Pad6) -> Net-(J4-Pad4)
- J5 pad 5: Net-(J4-Pad7) -> Net-(J4-Pad5)
- J5 pad 6: Net-(J4-Pad8) -> Net-(J4-Pad6)
- U1 pad 10: P1 -> SCL
- U1 pad 11: P2 -> ARD_RX
- U1 pad 12: P3 -> Net-(R2-Pad2)
- U1 pad 13: SCL -> P0
- U1 pad 14: SDA -> P1
- U1 pad 15: ARD_RX -> P2
- U1 pad 16: Net-(R2-Pad2) -> P3
- U1 pad 9: P0 -> SDA
Routing:
- net 5V: track 2.54 -> 98.4 mm, vias 0 -> 4
- net SDA: track 0.00 -> 87.7 mm
- net SCL: track 0.00 -> 72.6 mm, vias 0 -> 1
- net GND: track 5.08 -> 55.3 mm, vias 0 -> 4
- net ARD_RX: track 0.00 -> 37.4 mm
- net Net-(R1-Pad2): track 0.00 -> 34.3 mm, vias 0 -> 2
- net ICSPCLK: track 0.00 -> 33.9 mm
- net ARD_TX: track 0.00 -> 27.7 mm
- net ICSPDAT: track 0.00 -> 27.6 mm
- net INPUT_A: track 0.00 -> 25.7 mm
- net 3.3V: track 2.54 -> 25.0 mm, vias 0 -> 2
- net MCLR: track 0.00 -> 21.6 mm, vias 0 -> 2
- net INPUT_B: track 0.00 -> 20.8 mm
- net Net-(R2-Pad2): track 0.00 -> 13.0 mm
- net P0: track 0.00 -> 13.0 mm
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Other:
- board text added: "5V"
- board text added: "P0"
- board text added: "P1"
- board text added: "P2"
- board text added: "P3"
- board text added: "P4"
- board text added: "P5"
- board text added: "SCL"
- board text added: "SDA"

Commit message: Bugfix Arduino-Shield PCB
Parts:
- D1: footprint Diode_SMD:D_SOD-123 -> Footprints:SOD-80_HandSolder
- moved R3 2.55 mm to (146.7, 78.7), turned to 90 degrees
- moved U2 2.29 mm to (149.2, 92.1)
- moved R4 2.01 mm to (151.8, 80.0), turned to 270 degrees
- moved D1 2.01 mm to (149.2, 79.4), turned to 90 degrees
- moved C3 1.91 mm to (154.3, 80.0), turned to 270 degrees
Routing:
- net Earth: track 1.51 -> 5.11 mm, vias 1 -> 3
- net Net-(D1-Pad2): track 7.70 -> 5.81 mm
- net 3.3V: track 25.0 -> 26.9 mm
- net GND: track 55.3 -> 57.2 mm, vias 4 -> 7
- net Net-(U2-Pad1): track 0.00 -> 1.35 mm
- net Net-(C4-Pad1): track 3.98 -> 5.33 mm
- net INPUT_A: track 25.7 -> 26.5 mm
- net Net-(R3-Pad1): track 3.56 -> 4.24 mm
- net Net-(C3-Pad1): track 12.4 -> 12.9 mm

Commit message: Bugfix Arduino-Shield Schematic and PCB
Parts:
- added R7: 180, Resistor_SMD:R_0805_2012Metric_Pad1.15x1.40mm_HandSolder, F.Cu at (135.3, 69.2)
- added R8: 180, Resistor_SMD:R_0805_2012Metric_Pad1.15x1.40mm_HandSolder, F.Cu at (155.6, 99.1)
- added R9: 180, Resistor_SMD:R_0805_2012Metric_Pad1.15x1.40mm_HandSolder, F.Cu at (155.6, 91.4)
- R5, R6: value 10K -> 2K2
- moved C1 0.63 mm to (138.4, 91.4)
- moved C2 0.63 mm to (138.4, 89.5)
- moved R2 0.39 mm to (135.3, 66.7)
Connections:
- C3 pad 2: Earth -> GND
- U1 pad 11: ARD_RX -> Net-(R7-Pad2)
- U1 pad 5: INPUT_A -> Net-(R8-Pad1)
- U1 pad 6: INPUT_B -> Net-(R9-Pad1)
Routing:
- net Net-(R8-Pad1): track 0.00 -> 24.1 mm
- net INPUT_A: track 26.5 -> 5.40 mm
- net Net-(R9-Pad1): track 0.00 -> 18.1 mm
- net INPUT_B: track 20.8 -> 5.40 mm
- net Net-(R7-Pad2): track 0.00 -> 7.62 mm
- net ARD_RX: track 37.4 -> 31.7 mm
- net Earth: track 5.11 -> 0.00 mm, vias 3 -> 0
- net 5V: track 98.4 -> 99.8 mm
- net 3.3V: track 26.9 -> 26.2 mm
- net GND: track 57.2 -> 56.7 mm, vias 7 -> 9
Other:
- board text added: "A"
- board text added: "B"
- board text added: "PICUINO FREQUENCY COUNTER 04/2020"
- board text added: "ZCD"
