File: arduino_shield/kicad/freqcounter.sch (KiCad schematic (older format))
At the start: 34 parts, among them J1 ICSP PICKIT, J10 INPUT_A, J11 INPUT_B, J12 INPUT_ZCD, J13 I2C_1, J14 I2C_2, J15 PARALEL, J16 Ext_Clk, J2 Arduino_Power, J3 Arduino_Power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

Commit message: Updated Arduino-Shield Schematic and PCB
Parts:
- C4: value 100nF -> 1nF
Changed lines of the file:
@@
 P 7350 4000
 F 0 "C4" V 7500 3950 50  0000 L CNN
-F 1 "100nF" V 7200 3850 50  0000 L CNN
+F 1 "1nF" V 7200 3950 50  0000 L CNN
 F 2 "Capacitor_SMD:C_0805_2012Metric_Pad1.15x1.40mm_HandSolder" H 7388 3850 50  0001 C CNN
 F 3 "~" H 7350 4000 50  0001 C CNN

Commit message: Updated schematic and PCB with LCD connector
Parts:
- J15: value PARALEL -> LCD
Connections:
- net P0: no longer J15.7 (Pin_7)
- net P1: no longer J15.6 (Pin_6)
- net P2: no longer J15.5 (Pin_5)
- net P3: no longer J15.4 (Pin_4)
- net ICSPCLK renamed D6
- net ICSPDAT renamed D7
- new net D4: J15.5 (Pin_5)
- new net D5: J15.4 (Pin_4)
- new net E: J15.6 (Pin_6)
- new net RS: J15.7 (Pin_7)
Changed lines of the file:
@@
 Text GLabel 7200 3000 2    40   Input ~ 0
 P1
-Text GLabel 9100 5200 2    40   Input ~ 0
-P3
-Text GLabel 9100 5300 2    40   Input ~ 0
-P2
+Text GLabel 9700 5000 0    40   Input ~ 0
+D7
+Text GLabel 9700 5100 0    40   Input ~ 0
+D6
 Text GLabel 9100 5500 2    40   Input ~ 0
-P0
+RS
 Text GLabel 9100 5400 2    40   Input ~ 0
-P1
+E
 Text GLabel 9100 5600 2    40   Input ~ 0
 GND
@@
 P 8800 5200
 F 0 "J15" H 8900 5750 50  0000 C CNN
-F 1 "PARALEL" H 8900 5650 50  0000 C CNN
+F 1 "LCD" H 8900 5650 50  0000 C CNN
 F 2 "Footprints:Connector_1x08" H 8800 5200 50  0001 C CNN
 F 3 "~" H 8800 5200 50  0001 C CNN
@@
 	1    0    0    -1
 $EndComp
-Text GLabel 9100 5000 2    40   Input ~ 0
+Text GLabel 9900 5000 2    40   Input ~ 0
 ICSPDAT
-Text GLabel 9100 5100 2    40   Input ~ 0
+Text GLabel 9900 5100 2    40   Input ~ 0
 ICSPCLK
 Wire Wire Line
@@
 	8200 4000 8100 4000
 Connection ~ 8100 4000
+Text GLabel 9100 5200 2    40   Input ~ 0
+D5
+Text GLabel 9100 5300 2    40   Input ~ 0
+D4
+Text GLabel 9100 5000 2    40   Input ~ 0
+D7
+Text GLabel 9100 5100 2    40   Input ~ 0
+D6
+Wire Wire Line
+	9700 5100 9900 5100
+Wire Wire Line
+	9700 5000 9900 5000
 $EndSCHEMATC

Commit message: Bugfix schematic and PCB with LCD connector
Connections:
- net P0 is gone; now on net RS: U1.13 (RB4)
- net P1 is gone; now on net E: U1.14 (RC2)
- net P2 is gone; now on net D4: U1.15 (RC1)
- net P3 is gone; now on net D5: U1.16 (RC0)
Changed lines of the file:
@@
 SDA
 Text GLabel 7200 2800 2    40   Input ~ 0
-P3
+D5
 Text GLabel 7200 2900 2    40   Input ~ 0
-P2
+D4
 Text GLabel 7200 3100 2    40   Input ~ 0
-P0
+RS
 Text GLabel 7200 3000 2    40   Input ~ 0
-P1
+E
 Text GLabel 9700 5000 0    40   Input ~ 0
 D7
